File: tests/fixtures/sch_edit/edit.kicad_sch (KiCad schematic)
At the start: 4 parts, among them U1 LM358

Commit message: feat(sch): sch edit connects and disconnects pins, names unnamed nets (#57)
connect draws a short wire out from a free pin and what names the net at
its end -- a label, a global label, a power symbol like the net's others
-- where it touches nothing else. disconnect removes the wire from the pin
as far as it served the pin alone; what named the rest moves to where the
wire met it. rename of an unnamed net puts a label on one of its pins.
Changes are made in order, each on the design as the previous ones left
it, and the read-back holds the result to the expected partition of pins.
Parts:
- added R4, R5: 1k, symbol fixture:R
Connections:
- new net: R4.2, R5.2
- no-connect marks 5 -> 7
Changed lines of the file:
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@@
+	)
+	(symbol
+		(lib_id "fixture:R")
+		(at 50.8 76.2 0)
+		(unit 1)
+		(exclude_from_sim no)
+		(in_bom yes)
+		(on_board yes)
+		(dnp no)
+		(property "Reference" "R4"
+			(at 53.34 74.93 0)
+			(effects
+				(font
+					(size 1.27 1.27)
+				)
+			)
+		)
+		(property "Value" "1k"
+			(at 53.34 77.47 0)
+			(effects
+				(font
+					(size 1.27 1.27)
+				)
+			)
+		)
+		(property "Footprint" ""
+			(at 50.8 76.2 0)
+			(hide yes)
+			(effects
+				(font
+					(size 1.27 1.27)
+				)
+			)
+		)
+		(property "Datasheet" ""
+			(at 50.8 76.2 0)
+			(hide yes)
+			(effects
+				(font
+					(size 1.27 1.27)
+				)
+			)
+		)
+		(property "Description" ""
+			(at 50.8 76.2 0)
+			(hide yes)
+			(effects
+				(font
+					(size 1.27 1.27)
+				)
+			)
+		)
+		(pin "1"
+		)
+		(pin "2"
+		)
+		(instances
+			(project "edit"
+				(path "/580ac6fe-81b6-53f3-8b01-c074a56f485a"
+					(reference "R4")
+					(unit 1)
+				)
+			)
+		)
+	)
+	(symbol
+		(lib_id "fixture:R")
+		(at 63.5 76.2 0)
+		(unit 1)
+		(exclude_from_sim no)
+		(in_bom yes)
+		(on_board yes)
+		(dnp no)
+		(property "Reference" "R5"
+			(at 66.04 74.93 0)
+			(effects
+				(font
+					(size 1.27 1.27)
+				)
+			)
+		)
+		(property "Value" "1k"
+			(at 66.04 77.47 0)
+			(effects
+				(font
+					(size 1.27 1.27)
+				)
+			)
+		)
+		(property "Footprint" ""
+			(at 63.5 76.2 0)
+			(hide yes)
+			(effects
+				(font
+					(size 1.27 1.27)
+				)
+			)
+		)
+		(property "Datasheet" ""
+			(at 63.5 76.2 0)
+			(hide yes)
+			(effects
+				(font
+					(size 1.27 1.27)
+				)
+			)
+		)
+		(property "Description" ""
+			(at 63.5 76.2 0)
+			(hide yes)
+			(effects
+				(font
+					(size 1.27 1.27)
+				)
+			)
+		)
+		(pin "1"
+		)
+		(pin "2"
+		)
+		(instances
+			(project "edit"
+				(path "/580ac6fe-81b6-53f3-8b01-c074a56f485a"
+					(reference "R5")
+					(unit 1)
+				)
+			)
+		)
+	)
+	(no_connect
+		(at 50.8 72.39)
+	)
+	(no_connect
+		(at 63.5 72.39)
+	)
+	(wire
+		(pts
+			(xy 50.8 80.01) (xy 50.8 82.55)
+		)
+		(stroke
+			(width 0)
+			(type default)
+		)
+	)
+	(wire
+		(pts
+			(xy 50.8 82.55) (xy 63.5 82.55)
+		)
+		(stroke
+			(width 0)
+			(type default)
+		)
+	)
+	(wire
+		(pts
+			(xy 63.5 82.55) (xy 63.5 80.01)
+		)
+		(stroke
+			(width 0)
+			(type default)
+		)
 	)
 	(symbol

Commit message: feat(board): board update carries the schematic onto its board
What KiCad's Update PCB from Schematic does with its dialog's defaults,
in this process: parts matched to footprints by uuid path; references,
values, fields and DNP/BOM marks updated; a part naming another footprint
gets it from the project's libraries where the old one was; every pad on
its pin's net; a renamed net's tracks, vias and zones renamed with it.
New footprints wait beside the board; nothing is deleted; a footprint no
library has is passed over and said to be. The board is read back against
the schematic before it is written, and KiCad's own schematic-parity check
finds the updated fixture board true to its schematic.
Parts:
- R1, R2, R3, R4, R5: footprint (none) -> fixture:R_0805
- U1: footprint (none) -> fixture:SO8
Changed lines of the file:
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@@
 			)
 		)
-		(property "Footprint" ""
+		(property "Footprint" "fixture:R_0805"
 			(at 50.8 50.8 0)
 			(hide yes)
@@
 			)
 		)
-		(property "Footprint" ""
+		(property "Footprint" "fixture:R_0805"
 			(at 63.5 50.8 0)
 			(hide yes)
@@
 			)
 		)
-		(property "Footprint" ""
+		(property "Footprint" "fixture:R_0805"
 			(at 76.2 50.8 0)
 			(hide yes)
@@
 			)
 		)
-		(property "Footprint" ""
+		(property "Footprint" "fixture:SO8"
 			(at 101.6 50.8 0)
 			(hide yes)
@@
 			)
 		)
-		(property "Footprint" ""
+		(property "Footprint" "fixture:R_0805"
 			(at 50.8 76.2 0)
 			(hide yes)
@@
 			)
 		)
-		(property "Footprint" ""
+		(property "Footprint" "fixture:R_0805"
 			(at 63.5 76.2 0)
 			(hide yes)
@@
 			)
 		)
-		(property "Footprint" ""
+		(property "Footprint" "fixture:SO8"
 			(at 101.6 76.2 0)
 			(hide yes)
