File: tests/fixtures/sch_edit/edit_child.kicad_sch (KiCad schematic)
At the start: 2 parts

Commit message: feat(sch): sch edit connects and disconnects pins, names unnamed nets (#57)
connect draws a short wire out from a free pin and what names the net at
its end -- a label, a global label, a power symbol like the net's others
-- where it touches nothing else. disconnect removes the wire from the pin
as far as it served the pin alone; what named the rest moves to where the
wire met it. rename of an unnamed net puts a label on one of its pins.
Changes are made in order, each on the design as the previous ones left
it, and the read-back holds the result to the expected partition of pins.
Parts:
- added R11: 10k, symbol fixture:R
Connections:
- no-connect marks 0 -> 2
Changed lines of the file:
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@@
 		)
+	)
+	(symbol
+		(lib_id "fixture:R")
+		(at 88.9 50.8 0)
+		(unit 1)
+		(exclude_from_sim no)
+		(in_bom yes)
+		(on_board yes)
+		(dnp no)
+		(property "Reference" "R11"
+			(at 91.44 49.53 0)
+			(effects
+				(font
+					(size 1.27 1.27)
+				)
+			)
+		)
+		(property "Value" "10k"
+			(at 91.44 52.07 0)
+			(effects
+				(font
+					(size 1.27 1.27)
+				)
+			)
+		)
+		(property "Footprint" ""
+			(at 88.9 50.8 0)
+			(hide yes)
+			(effects
+				(font
+					(size 1.27 1.27)
+				)
+			)
+		)
+		(property "Datasheet" ""
+			(at 88.9 50.8 0)
+			(hide yes)
+			(effects
+				(font
+					(size 1.27 1.27)
+				)
+			)
+		)
+		(property "Description" ""
+			(at 88.9 50.8 0)
+			(hide yes)
+			(effects
+				(font
+					(size 1.27 1.27)
+				)
+			)
+		)
+		(pin "1"
+		)
+		(pin "2"
+		)
+		(instances
+			(project "edit"
+				(path "/580ac6fe-81b6-53f3-8b01-c074a56f485a/43040844-219b-5afe-956b-f02b17d3693a"
+					(reference "R11")
+					(unit 1)
+				)
+				(path "/580ac6fe-81b6-53f3-8b01-c074a56f485a/cc4316f9-1336-533b-887c-887029e43744"
+					(reference "R21")
+					(unit 1)
+				)
+			)
+		)
+	)
+	(no_connect
+		(at 88.9 46.99)
+	)
+	(no_connect
+		(at 88.9 54.61)
 	)
 	(embedded_fonts no)

Commit message: feat(board): board update carries the schematic onto its board
What KiCad's Update PCB from Schematic does with its dialog's defaults,
in this process: parts matched to footprints by uuid path; references,
values, fields and DNP/BOM marks updated; a part naming another footprint
gets it from the project's libraries where the old one was; every pad on
its pin's net; a renamed net's tracks, vias and zones renamed with it.
New footprints wait beside the board; nothing is deleted; a footprint no
library has is passed over and said to be. The board is read back against
the schematic before it is written, and KiCad's own schematic-parity check
finds the updated fixture board true to its schematic.
Parts:
- C10, R10, R11: footprint (none) -> fixture:R_0805
Changed lines of the file:
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@@
 			)
 		)
-		(property "Footprint" ""
+		(property "Footprint" "fixture:R_0805"
 			(at 50.8 50.8 0)
 			(hide yes)
@@
 			)
 		)
-		(property "Footprint" ""
+		(property "Footprint" "fixture:R_0805"
 			(at 63.5 50.8 0)
 			(hide yes)
@@
 			)
 		)
-		(property "Footprint" ""
+		(property "Footprint" "fixture:R_0805"
 			(at 88.9 50.8 0)
 			(hide yes)
